Commit message: Added Camera Module 3

File: src/amr_robot/urdf/properties.xacro (robot description, xacro)
@@ -10,5 +10,5 @@
      <!-- Wheel Properties-->
   <xacro:property name="wheel_radius" value="0.034"/>
-  <xacro:property name="wheel_thickness" value="0.02"/>
+  <xacro:property name="wheel_thickness" value="0.05"/>
   <xacro:property name="wheel_mass" value="0.1"/>
   <xacro:property name="wheel_friction" value="1.0"/>
@@ -29,9 +29,10 @@
   <xacro:property name="lidar_y" value="0.0"/>
   <xacro:property name="lidar_z" value="0.072"/>
+  <xacro:property name="lidar_yaw" value="3.14159"/>
   <xacro:property name="lidar_frame" value="laser_frame"/>
       <!-- IMU - BN0085-->
   <xacro:property name="imu_x" value="0.0"/>
   <xacro:property name="imu_y" value="0.0"/>
-  <xacro:property name="imu_z" value="0.026"/>
+  <xacro:property name="imu_z" value="0.068"/>
       <!-- IR -->
   <xacro:property name="ir_x" value="0.076"/>

File: src/amr_robot/urdf/sensors.xacro (robot description, xacro)
@@ -8,5 +8,5 @@
     <origin
       xyz="${lidar_x} ${lidar_y} ${lidar_z}"
-      rpy="0.0 0.0 0.0" />
+      rpy="0.0 0.0 ${lidar_yaw}" />
   </joint>
   <link name="laser_frame">

File: src/amr_robot/urdf/wheels.xacro (robot description, xacro)
@@ -6,9 +6,4 @@
       <parent link="base_link" />
       <child link="${prefix}_wheel" />
-      <!-- Correct placement:
-           - x = 0
-           - y = ± wheel_y_offset (left/right)
-           - z = 0          (wheel center is at base_link height)
-           - rpy = -pi/2 0 0  → cylinder axis becomes horizontal (along Y) -->
       <origin
         xyz="${wheel_x_offset} ${y_reflect * wheel_y_offset} 0.0"
